File: hardware/KEMOJO.kicad_pcb (KiCad board)
At the start: 4 copper layers, 101.6 x 55.9 mm, 28 parts, among them J1 Conn_02x03_Odd_Even, J10 Conn_02x02_Counter_Clockwise, J11 Conn_01x40, J12 Conn_02x02_Odd_Even, J2 DE9_Plug, J3 DE9_Plug, J4 Mini-DIN-6, J5 Mini-DIN-6, J6 Conn_01x06_Pin, J7 Conn_02x04_Odd_Even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

Commit message: Add more documentation.
Other:
- board text added: "7.3728 MHz"
- board text added: "Keyboard/mouse/joystick controller for RCBUS, version V1B © 2024 Rob Gowin github.com/codesmythe/KEMOJO"
- board text added: "Licensed under CC-BY-NC-SA 4.0"
- board text removed: "7.3728 MHz MHz"
- board text removed: "JLCJLCJLCJLC"
- board text removed: "Keyboard/mouse/joystick controller for RCBUS, version V1A © 2024 Rob Gowin."
Changed lines of the file:
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@@
 	(title_block
 		(title "KEMOJO")
-		(date "2024-11-29")
-		(rev "V1A")
+		(date "2025-06-12")
+		(rev "V1B")
 		(comment 1 "Licensed under CC-BY-NC-SA 4.0")
 	)
@@
 			(drillshape 0)
 			(scaleselection 1)
-			(outputdirectory "KEMOJO_V1A")
+			(outputdirectory "KEMOJO_V1B")
 		)
 	)
@@
 			)
 		)
-		(property "Mouser PN" "575-944424"
-			(at 0 0 0)
-			(unlocked yes)
-			(layer "F.Fab")
-			(hide yes)
-			(effects
-				(font
-					(size 1 1)
-					(thickness 0.15)
-				)
-			)
-		)
 		(sheetfile "KEMOJO.kicad_sch")
 		(attr through_hole)
@@
 		(tags "to-92 sc-43 sc-43a sot54 PA33 transistor")
 		(property "Reference" "Q1"
-			(at 1.27 -4.4 0)
+			(at -2.7432 -2.3172 0)
 			(layer "F.SilkS")
 			(effects
@@
 		)
 	)
-	(gr_text "7.3728 MHz\nMHz"
+	(gr_text "7.3728\nMHz"
 		(at 195.637 131.732676 0)
 		(layer "F.SilkS")
@@
 		)
 	)
-	(gr_text "Keyboard/mouse/joystick controller\nfor RCBUS, version V1A\n© 2024 Rob Gowin."
-		(at 210.7826 138.7992 0)
+	(gr_text "Keyboard/mouse/joystick controller\nfor RCBUS, version V1B\n© 2024 Rob Gowin\ngithub.com/codesmythe/KEMOJO"
+		(at 210.9096 140.3232 0)
 		(layer "F.SilkS")
 		(effects
@@
 		)
 	)
-	(gr_text "JLCJLCJLCJLC"
-		(at 173.4586 144.2952 0)
+	(gr_text "IEx\nBYPASS"
+		(at 234.8286 143.5652 0)
 		(layer "F.SilkS")
 		(effects
@@
 				(thickness 0.15)
 			)
-			(justify left bottom)
+			(justify bottom)
 		)
 	)
-	(gr_text "IEx\nBYPASS"
-		(at 234.8286 143.5652 0)
+	(gr_text "Licensed under CC-BY-NC-SA 4.0"
+		(at 158.5468 152.8572 0)
 		(layer "F.SilkS")
 		(effects
@@
 				(thickness 0.15)
 			)
-			(justify bottom)
+			(justify left bottom)
 		)
 	)
