File: hardware/KEMOJO.kicad_sch (KiCad schematic)
At the start: 27 parts, among them J1 Conn_02x03_Odd_Even, J10 Conn_02x02_Counter_Clockwise, J11 Conn_01x40, J12 Conn_02x02_Odd_Even, J2 DE9_Plug, J3 DE9_Plug, J4 Mini-DIN-6, J5 Mini-DIN-6, J6 Conn_01x06_Pin, J7 Conn_02x04_Odd_Even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

Commit message: Add more documentation.
Parts:
- C1, C2, C3, C4, C5: PartNum00 (none) -> 594-K104K15X7RF5WH5; PartVendor00 (none) -> Mouser
- D1: PartNum00 (none) -> 859-LTL-4251N; PartVendor00 (none) -> Mouser
- J1: PartNum00 (none) -> 200-TSW10307TD; PartVendor00 (none) -> Mouser
- J10, J12: PartNum00 (none) -> 200-TSW10207TD; PartVendor00 (none) -> Mouser
- J11: PartNum00 (none) -> 710-61304011021; PartVendor00 (none) -> Mouser
- J2, J3: PartNum00 (none) -> 523-L7SDE9PA4CH4RC39; PartVendor00 (none) -> Mouser
- J4, J5: PartNum00 (none) -> 490-MD-40SM; PartVendor00 (none) -> Mouser
- J6: PartNum00 (none) -> 737-PH1RB-06-UA; PartVendor00 (none) -> Mouser
- J7, J8: PartNum00 (none) -> 200-TSW10407TD; PartVendor00 (none) -> Mouser
- J9: PartNum00 (none) -> 200-TSW10807TD; PartVendor00 (none) -> Mouser
- JP4: PartNum00 (none) -> 200-TSW10207TS; PartVendor00 (none) -> Mouser
- Q1: PartNum00 (none) -> 512-2N7000; PartVendor00 (none) -> Mouser
- R11: PartNum00 (none) -> 603-MFR-25FTF52-470R; PartVendor00 (none) -> Mouser
- U1: PartNum00 (none) -> 556-ATMEGA328P-PU; PartNum01 (none) -> 737-ICS-328-T; PartVendor00 (none) -> Mouser; PartVendor01 (none) -> Mouser
- U2: Mouser PN 595-TL16C550CFNR -> (none); Mouser PN 2 575-944424 -> (none); PartNum00 (none) -> 595-TL16C550CFNR; PartNum01 (none) -> 575-944424; PartVendor00 (none) -> Mouser; PartVendor01 (none) -> Mouser
- U3: PartNum00 (none) -> 595-SN74LS138NE4; PartNum01 (none) -> 571-1-2199298-4; PartVendor00 (none) -> Mouser; PartVendor01 (none) -> Mouser
- U4: PartNum00 (none) -> 595-SN74LS04NE4; PartNum01 (none) -> 571-1-2199298-3; PartVendor00 (none) -> Mouser; PartVendor01 (none) -> Mouser
- X1: PartNum00 (none) -> 774-MXO45HS-3C-7.3; PartNum01 (none) -> 535-1108800; PartVendor00 (none) -> Mouser; PartVendor01 (none) -> Mouser
